File: picoRemote/board/dmx-remote.kicad_pcb (KiCad board)
At the start: 2 copper layers, 62.5 x 51.5 mm, 17 parts, among them J1 multiplexer control, J10 power, J2 multiplexer in, J3 inputs, J4 vcc inputs, J5 gnd inputs, J6 oled, J7 nunchuck, J8 RF, J9 DMX, M1 Module_RaspberryPi_PicoW_Comb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

Commit message: edited transmitter and receiver for animallove.
Parts:
- added C5: 100n, fab:C_1206, F.Cu at (84.4, 88.2)
- added C6: 100n, fab:C_1206, F.Cu at (92.4, 96.0)
- added J11: Conn_01x04, Connector_PinHeader_2.54mm:PinHeader_1x04_P2.54mm_Vertical, F.Cu at (130.3, 85.0)
- added J12: Conn_01x04, Connector_PinHeader_2.54mm:PinHeader_1x04_P2.54mm_Vertical, F.Cu at (132.9, 85.0)
- added J13: Conn_01x04, Connector_PinHeader_2.54mm:PinHeader_1x04_P2.54mm_Vertical, F.Cu at (132.9, 96.2)
- added J14: Conn_01x04, Connector_PinHeader_2.54mm:PinHeader_1x04_P2.54mm_Vertical, F.Cu at (132.9, 107.4)
- added J15: Conn_01x04, Connector_PinHeader_2.54mm:PinHeader_1x04_P2.54mm_Vertical, F.Cu at (132.9, 118.6)
- added J16: Conn_01x04, Connector_PinHeader_2.54mm:PinHeader_1x04_P2.54mm_Vertical, F.Cu at (135.4, 85.0)
- added J17: Conn_01x04, Connector_PinHeader_2.54mm:PinHeader_1x04_P2.54mm_Vertical, F.Cu at (135.4, 96.2)
- added J18: Conn_01x04, Connector_PinHeader_2.54mm:PinHeader_1x04_P2.54mm_Vertical, F.Cu at (135.4, 107.4)
- added J19: Conn_01x04, Connector_PinHeader_2.54mm:PinHeader_1x04_P2.54mm_Vertical, F.Cu at (135.4, 118.6)
- added J20: grove-ENCODER, Connector:NS-Tech_Grove_1x04_P2mm_Vertical, F.Cu at (75.0, 94.2)
- added J21: ELRS-out, Connector_PinHeader_2.54mm:PinHeader_1x03_P2.54mm_Vertical, F.Cu at (81.2, 80.8)
- added J22: keypad, Connector_PinHeader_2.54mm:PinHeader_1x09_P2.54mm_Vertical, F.Cu at (82.9, 107.8)
- added JP1: bypass, Jumper:SolderJumper-2_P1.3mm_Open_Pad1.0x1.5mm, B.Cu at (84.4, 80.4)
- added R2: 10k, fab:R_1206, F.Cu at (96.8, 101.3)
- added R3: 10k, fab:R_1206, F.Cu at (96.8, 91.1)
- added R4: 10k, fab:R_1206, F.Cu at (96.9, 88.4)
- added R5: 4k7, fab:R_1206, B.Cu at (78.0, 106.0)
- added R6: 4k7, fab:R_1206, B.Cu at (78.0, 111.6)
- added R7: 4k7, fab:R_1206, B.Cu at (78.1, 98.9)
- added R8: 4k7, fab:R_1206, B.Cu at (78.0, 93.4)
- added RN1: 10k, Resistor_THT:R_Array_SIP5, F.Cu at (109.0, 127.1)
- added RN2: 10k, Resistor_THT:R_Array_SIP5, F.Cu at (109.1, 123.7)
- added RN3: 10k, Resistor_THT:R_Array_SIP5, F.Cu at (109.1, 120.4)
- added RN4: 10k, Resistor_THT:R_Array_SIP5, F.Cu at (109.1, 117.1)
- added RN5: 10k, Resistor_THT:R_Array_SIP5, F.Cu at (109.2, 92.4)
- added RN6: 10k, Resistor_THT:R_Array_SIP5, F.Cu at (109.2, 89.1)
- added RN7: 10k, Resistor_THT:R_Array_SIP5, F.Cu at (109.2, 85.8)
- added RN8: 10k, Resistor_THT:R_Array_SIP5, F.Cu at (109.2, 82.4)
- added U2: 74LVC2G241, Package_SO:SSOP-8_3.9x5.05mm_P1.27mm, F.Cu at (96.6, 96.2)
- J3: value inputs -> Conn_01x04; footprint Connector_PinHeader_2.54mm:PinHeader_1x16_P2.54mm_Vertical -> Connector_PinHeader_2.54mm:PinHeader_1x04_P2.54mm_Vertical
- J4: value vcc inputs -> Conn_01x04; footprint Connector_PinHeader_2.54mm:PinHeader_1x16_P2.54mm_Vertical -> Connector_PinHeader_2.54mm:PinHeader_1x04_P2.54mm_Vertical
- J5: value gnd inputs -> Conn_01x04; footprint Connector_PinSocket_2.54mm:PinSocket_1x16_P2.54mm_Vertical -> Connector_PinHeader_2.54mm:PinHeader_1x04_P2.54mm_Vertical
- J6: value oled -> grove-OLED; footprint Connector_JST:JST_XH_B4B-XH-A_1x04_P2.50mm_Vertical -> Connector:NS-Tech_Grove_1x04_P2mm_Vertical
- J7: value nunchuck -> JST-nunchuck
- J8: value RF -> JST-RF
- J9: value DMX -> grove-serial; footprint Connector_JST:JST_XH_B4B-XH-A_1x04_P2.50mm_Vertical -> Connector:NS-Tech_Grove_1x04_P2mm_Vertical
- moved J6 560.4 mm to (81.6, 94.2), turned to 0 degrees
- moved D1 552.8 mm to (74.3, 89.2), turned to 180 degrees
- moved R1 549.5 mm to (80.2, 89.2), turned to 0 degrees
- moved J10 547.9 mm to (75.5, 81.9), turned to -90 degrees
- moved J2 515.0 mm to (126.0, 85.7)
- moved J8 512.8 mm to (74.2, 127.1)
- moved J7 512.3 mm to (74.3, 113.5)
- moved J5 511.4 mm to (130.4, 118.6)
- moved J1 510.7 mm to (110.6, 95.9)
- moved J4 510.1 mm to (130.4, 107.4)
- moved C1 508.8 mm to (134.3, 81.6)
- moved C2 508.3 mm to (80.0, 127.2), turned to -90 degrees
- moved M1 508.2 mm to (96.8, 104.3)
- moved C4 507.6 mm to (79.9, 113.8), turned to -90 degrees
- moved C3 504.8 mm to (81.7, 104.0)
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Connections:
- J2 pad 1: Net-(J2-Pin_1) -> Net-(J11-Pin_1)
- J2 pad 2: Net-(J2-Pin_2) -> Net-(J11-Pin_2)
- J2 pad 3: Net-(J2-Pin_3) -> Net-(J11-Pin_3)
- J2 pad 4: Net-(J2-Pin_4) -> Net-(J11-Pin_4)
- J3 pad 1: Net-(J2-Pin_1) -> Net-(J2-Pin_5)
- J3 pad 2: Net-(J2-Pin_2) -> Net-(J2-Pin_6)
- J3 pad 3: Net-(J2-Pin_3) -> Net-(J2-Pin_7)
- J3 pad 4: Net-(J2-Pin_4) -> Net-(J2-Pin_8)
- J4 pad 1: +3.3V -> Net-(J2-Pin_9)
- J4 pad 2: +3.3V -> Net-(J2-Pin_10)
- J4 pad 3: +3.3V -> Net-(J2-Pin_11)
- J4 pad 4: +3.3V -> Net-(J2-Pin_12)
- J5 pad 1: GND -> Net-(J2-Pin_13)
- J5 pad 2: GND -> Net-(J2-Pin_14)
- J5 pad 3: GND -> Net-(J2-Pin_15)
- J5 pad 4: GND -> Net-(J2-Pin_16)
- J6 pad 1: GND -> /SCL1
- J6 pad 2: +3.3V -> /SDA1
- J6 pad 3: /SCL -> +3.3V
- J6 pad 4: /SDA -> GND
- J8 pad 3: /RF-RxD -> /DMX-RxD
- J8 pad 4: /RF-TxD -> /DMX-TxD
- J9 pad 1: GND -> /RF-TxD
- J9 pad 2: +3.3V -> /RF-RxD
- J9 pad 3: /DMX-RxD -> +3.3V
- J9 pad 4: /DMX-TxD -> GND
- M1 pad 1: /DMX-RxD -> /RF-RxD
- M1 pad 10: unconnected-(M1-GP7-Pad10) -> /SCL1
- M1 pad 11: /RF-RxD -> /DMX-RxD
- M1 pad 12: /RF-TxD -> /DMX-TxD
- M1 pad 14: unconnected-(M1-GP10-Pad14) -> /RF-S/R
- M1 pad 15: unconnected-(M1-GP11-Pad15) -> /COL3
- M1 pad 16: unconnected-(M1-GP12-Pad16) -> /ROW1
- M1 pad 17: unconnected-(M1-GP13-Pad17) -> /ROW2
- M1 pad 19: unconnected-(M1-GP14-Pad19) -> /ROW3
- M1 pad 2: /DMX-TxD -> /RF-TxD
- M1 pad 20: unconnected-(M1-GP15-Pad20) -> /ROW4
- M1 pad 4: unconnected-(M1-GP2-Pad4) -> /COL1
- M1 pad 5: unconnected-(M1-GP3-Pad5) -> /COL2
- M1 pad 9: unconnected-(M1-GP6-Pad9) -> /SDA1
Routing:
- net +3.3V: track 161.9 -> 262.7 mm, vias 0 -> 1
- net GND: track 224.2 -> 285.9 mm
- net Net-(J21-Pin_1): track 0.00 -> 37.0 mm
- net /SCL: track 59.6 -> 22.9 mm
- net /SDA: track 55.8 -> 22.9 mm
- net /COL1: track 0.00 -> 32.5 mm
- net +5V: track 16.6 -> 45.6 mm
- net /RF-S/R: track 0.00 -> 29.0 mm
- net Net-(J11-Pin_4): track 0.00 -> 25.8 mm
- net /COL2: track 0.00 -> 24.0 mm
- net Net-(J2-Pin_9): track 4.33 -> 27.3 mm
- net Net-(J2-Pin_8): track 4.33 -> 26.8 mm
- net Net-(J2-Pin_13): track 4.33 -> 26.8 mm
- net /SCL1: track 0.00 -> 22.4 mm
- net Net-(J11-Pin_3): track 0.00 -> 22.2 mm
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Other:
- board size 62.5 x 51.5 mm -> 67 x 52 mm
- board text added: "- + C D"
- board text added: "- + D C"
- board text added: "- + S"
- board text added: "- + Tx Rx"
- board text added: "5V - +"
- board text added: "Rx Tx + -"
- board text added: "S + -"
- board text added: "UART0"
- board text added: "in1"
- board text added: "in16"
- board text added: "keypad"
- board text added: "optional half- duplex driver for ELRS module"
- board text added: "picoRemote E13 2025"
- board text added: "rn8 UP 1-4 rn7 DOWN 1-4 rn6 UP 5-8 rn5 DOWN 5-8 rn4 UP 9-12 rn3 DOWN 9-12 rn2 UP 13-16 rn1 DOWN 13-16"
- board text added: "there is a solder jumper on the bot lyr for bypass"
