File: picoRemote/board/dmx-remote.kicad_sch (KiCad schematic)
At the start: 17 parts, among them J1 multiplexer control, J10 power, J2 multiplexer in, J3 inputs, J4 vcc inputs, J5 gnd inputs, J6 oled, J7 nunchuck, J8 RF, J9 DMX, M1 Module_RaspberryPi_PicoW_Comb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

Commit message: edited transmitter and receiver for animallove.
Parts:
- removed J3: inputs, Connector_PinHeader_2.54mm:PinHeader_1x16_P2.54mm_Vertical, symbol Connector_Generic:Conn_01x16
- removed J4: vcc inputs, Connector_PinHeader_2.54mm:PinHeader_1x16_P2.54mm_Vertical, symbol Connector_Generic:Conn_01x16
- removed J5: gnd inputs, Connector_PinSocket_2.54mm:PinSocket_1x16_P2.54mm_Vertical, symbol Connector_Generic:Conn_01x16
- added C5, C6: 100n, fab:C_1206, symbol Device:C
- added J11, J12, J13, J14, J15, J16, J17, J18, J19, J3, J4, J5: Conn_01x04, Connector_PinHeader_2.54mm:PinHeader_1x04_P2.54mm_Vertical, symbol Connector_Generic:Conn_01x04
- added J20: grove-ENCODER, Connector:NS-Tech_Grove_1x04_P2mm_Vertical, symbol Connector_Generic:Conn_01x04
- added J21: ELRS-out, Connector_PinHeader_2.54mm:PinHeader_1x03_P2.54mm_Vertical, symbol Connector_Generic:Conn_01x03
- added J22: keypad, Connector_PinHeader_2.54mm:PinHeader_1x09_P2.54mm_Vertical, symbol Connector_Generic:Conn_01x09
- added JP1: bypass, Jumper:SolderJumper-2_P1.3mm_Open_Pad1.0x1.5mm, symbol Jumper:Jumper_2_Bridged
- added R2, R3, R4: 10k, fab:R_1206, symbol Device:R
- added R5, R6, R7, R8: 4k7, fab:R_1206, symbol Device:R
- added RN1, RN2, RN3, RN4, RN5, RN6, RN7, RN8: 10k, Resistor_THT:R_Array_SIP5, symbol Device:R_Network04
- added U2: 74LVC2G241, Package_SO:SSOP-8_3.9x5.05mm_P1.27mm, symbol 74xGxx:74LVC2G241
- J6: value oled -> grove-OLED; footprint Connector_JST:JST_XH_B4B-XH-A_1x04_P2.50mm_Vertical -> Connector:NS-Tech_Grove_1x04_P2mm_Vertical
- J7: value nunchuck -> JST-nunchuck
- J8: value RF -> JST-RF
- J9: value DMX -> grove-serial; footprint Connector_JST:JST_XH_B4B-XH-A_1x04_P2.50mm_Vertical -> Connector:NS-Tech_Grove_1x04_P2mm_Vertical
Connections:
- net +3.3V: now also J6.3 (Pin_3), J9.3 (Pin_3), C5.1, C6.1, J12.1 (Pin_1), J12.2 (Pin_2), J12.3 (Pin_3), J12.4 (Pin_4), J13.1 (Pin_1), J13.2 (Pin_2), J13.3 (Pin_3), J13.4 (Pin_4), J14.1 (Pin_1), J14.2 (Pin_2), J14.3 (Pin_3), J14.4 (Pin_4), J15.1 (Pin_1), J15.2 (Pin_2), J15.3 (Pin_3), J15.4 (Pin_4), J20.3 (Pin_3), R2.1, R3.1, R5.1, R6.1, R7.1, R8.1, RN2.1 (common), RN4.1 (common), RN6.1 (common), RN8.1 (common), U2.8 (VCC); no longer J6.2 (Pin_2), J9.2 (Pin_2)
- net +5V: now also J21.2 (Pin_2)
- net DMX-RxD: now also J8.3 (Pin_3), M1.11 (GP8); no longer J9.3 (Pin_3), M1.1 (GP0)
- net DMX-TxD: now also J8.4 (Pin_4), M1.12 (GP9); no longer J9.4 (Pin_4), M1.2 (GP1)
- net GND: now also J6.4 (Pin_4), J9.4 (Pin_4), C5.2, C6.2, J16.1 (Pin_1), J16.2 (Pin_2), J16.3 (Pin_3), J16.4 (Pin_4), J17.1 (Pin_1), J17.2 (Pin_2), J17.3 (Pin_3), J17.4 (Pin_4), J18.1 (Pin_1), J18.2 (Pin_2), J18.3 (Pin_3), J18.4 (Pin_4), J19.1 (Pin_1), J19.2 (Pin_2), J19.3 (Pin_3), J19.4 (Pin_4), J20.4 (Pin_4), J21.3 (Pin_3), R4.2, RN1.1 (common), RN3.1 (common), RN5.1 (common), RN7.1 (common), U2.4 (GND); no longer J6.1 (Pin_1), J9.1 (Pin_1)
- net RF-RxD: now also J9.2 (Pin_2), M1.1 (GP0), JP1.1 (A), U2.5; no longer J8.3 (Pin_3), M1.11 (GP8)
- net RF-TxD: now also J9.1 (Pin_1), M1.2 (GP1), R3.2, U2.6; no longer J8.4 (Pin_4), M1.12 (GP9)
- net SCL: now also R6.2; no longer J6.3 (Pin_3)
- net SDA: now also R5.2; no longer J6.4 (Pin_4)
- net at J2.1 (Pin_1): now also J11.1 (Pin_1), RN7.5 (R4), RN8.5 (R4)
- net at J2.10 (Pin_10): now also J4.2 (Pin_2), RN3.3 (R2), RN4.3 (R2)
- net at J2.11 (Pin_11): now also J4.3 (Pin_3), RN3.4 (R3), RN4.4 (R3)
- net at J2.12 (Pin_12): now also J4.4 (Pin_4), RN3.5 (R4), RN4.5 (R4)
- net at J2.13 (Pin_13): now also J5.1 (Pin_1), RN1.2 (R1), RN2.2 (R1)
- net at J2.14 (Pin_14): now also J5.2 (Pin_2), RN1.3 (R2), RN2.3 (R2)
- net at J2.15 (Pin_15): now also J5.3 (Pin_3), RN1.4 (R3), RN2.4 (R3)
- net at J2.16 (Pin_16): now also J5.4 (Pin_4), RN1.5 (R4), RN2.5 (R4)
- net at J2.2 (Pin_2): now also J11.2 (Pin_2), RN7.4 (R3), RN8.4 (R3)
- net at J2.3 (Pin_3): now also J11.3 (Pin_3), RN7.3 (R2), RN8.3 (R2)
- net at J2.4 (Pin_4): now also J11.4 (Pin_4), RN7.2 (R1), RN8.2 (R1)
- net at J2.5 (Pin_5): now also J3.1 (Pin_1), RN5.5 (R4), RN6.5 (R4)
- net at J2.6 (Pin_6): now also J3.2 (Pin_2), RN5.4 (R3), RN6.4 (R3)
- net at J2.7 (Pin_7): now also J3.3 (Pin_3), RN5.3 (R2), RN6.3 (R2)
- net at J2.8 (Pin_8): now also J3.4 (Pin_4), RN5.2 (R1), RN6.2 (R1)
- net at J2.9 (Pin_9): now also J4.1 (Pin_1), RN3.2 (R1), RN4.2 (R1)
- net SCL1: now reaches M1.10 (GP7)
- net SCL1: now also J6.1 (Pin_1), J20.1 (Pin_1), R8.2
- net RF-S/R: now reaches M1.14 (GP10)
- net RF-S/R: now also R4.1, U2.1, U2.7
- net COL3: now reaches M1.15 (GP11)
- net COL3: now also J22.6 (Pin_6)
- net ROW1: now reaches M1.16 (GP12)
- net ROW1: now also J22.3 (Pin_3)
- net ROW2: now reaches M1.17 (GP13)
- net ROW2: now also J22.8 (Pin_8)
- net ROW3: now reaches M1.19 (GP14)
- net ROW3: now also J22.7 (Pin_7)
- net ROW4: now reaches M1.20 (GP15)
- net ROW4: now also J22.5 (Pin_5)
- net COL1: now reaches M1.4 (GP2)
- net COL1: now also J22.4 (Pin_4)
- net COL2: now reaches M1.5 (GP3)
- net COL2: now also J22.2 (Pin_2)
- net SDA1: now reaches M1.9 (GP6)
- net SDA1: now also J6.2 (Pin_2), J20.2 (Pin_2), R7.2
- new net: J21.1 (Pin_1), JP1.2 (B), R2.2, U2.2, U2.3
Other:
- moved on the sheet: J2, J6, J9
