File: picoControl/board/kicadV3.0/smallcontrol.kicad_pcb (KiCad board)
At the start: 2 copper layers, 60.1 x 50.7 mm, 45 parts, among them J1 dynamixel, J10 OLED, J11 CSRF, J14 lineOut1, J15 grove I2C, J2 Audio1, J23 PowerIn, J24 grove GPIO / waveshare DDSM, J25 PowerIn, J26 grove GPIO / waveshare DDSM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

Commit message: update config.cpp system
Parts:
- added J16: grove Analog, Connector:NS-Tech_Grove_1x04_P2mm_Vertical, F.Cu at (94.8, 127.5)
- C1, C15, C2, C5, C8: footprint fab:C_1206 -> Capacitor_SMD:C_0603_1608Metric_Pad1.08x0.95mm_HandSolder
- J15, J24, J26: footprint Connectors:Grove_1x04 -> Connector:NS-Tech_Grove_1x04_P2mm_Vertical
- R1, R2, R3, R4: footprint fab:R_1206 -> Resistor_SMD:R_0603_1608Metric_Pad0.98x0.95mm_HandSolder
- R10, R9: footprint fab:R_1206 -> Resistor_SMD:R_0603_1608Metric_Pad0.98x0.95mm_HandSolder; moved to B.Cu
- moved C15 30.4 mm to (111.7, 100.8), turned to 180 degrees
- moved D1 22.0 mm to (115.2, 114.0)
- moved F1 21.7 mm to (121.0, 115.0), turned to -90 degrees
- moved C5 20.1 mm to (94.5, 114.3)
- moved C7 16.6 mm to (96.1, 102.2)
- moved U1 11.5 mm to (97.0, 117.0)
- moved R2 11.0 mm to (101.1, 117.0)
- moved R4 10.7 mm to (93.2, 117.2)
- moved R3 10.5 mm to (98.2, 114.3)
- moved J14 7.82 mm to (71.9, 106.7), turned to 0 degrees
- moved F2 6.10 mm to (101.0, 108.1)
- moved D2 6.10 mm to (94.3, 108.1)
- moved JP4 5.86 mm to (121.6, 122.6), turned to 180 degrees
- moved C8 5.12 mm to (77.6, 97.6), turned to 180 degrees
- moved J25 3.76 mm to (118.2, 108.5)
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Connections:
- J1 pad 1: GND -> /B
- J1 pad 2: /12Vfused -> /A
- J1 pad 3: /A -> /12Vfused
- J1 pad 4: /B -> GND
- J7 pad 2: /PWM1 -> +3.3V
- J7 pad 3: /INA1 -> /PWM1
- J7 pad 4: /INB1 -> /PWM2
- J7 pad 5: GND -> /INA1
- J7 pad 6: +3.3V -> /INB1
- J7 pad 7: /PWM2 -> /INA2
- J7 pad 8: /INA2 -> /INB2
- J7 pad 9: /INB2 -> GND
- M1 pad 20: /GP10 -> /GP15
- M1 pad 32: unconnected-(M1-GP27-Pad32) -> Net-(J16-Pin_4)
- M1 pad 34: unconnected-(M1-GP28-Pad34) -> Net-(J16-Pin_3)
- R2 pad 1: +5V -> +3.3V
- U1 pad 8: +5V -> +3.3V
Routing:
- net +5V: track 87.8 -> 30.1 mm, vias 15 -> 0
- net /PWM2: track 30.8 -> 67.5 mm
- net Net-(J16-Pin_3): track 0.00 -> 33.4 mm
- net Net-(J16-Pin_4): track 0.00 -> 27.5 mm
- net +12V: track 39.1 -> 66.3 mm, vias 2 -> 4
- net Net-(J3-Pin_1): track 45.4 -> 71.9 mm
- net /RFRX: track 26.2 -> 52.4 mm
- net /GP15: track 0.00 -> 25.2 mm
- net /12Vin: track 49.2 -> 27.5 mm, vias 1 -> 0
- net /RS485TX: track 26.4 -> 45.7 mm
- net /B: track 43.6 -> 24.5 mm, vias 1 -> 2
- net GND: track 312.1 -> 293.9 mm, vias 4 -> 2
- net /AX12SR: track 58.9 -> 40.9 mm, vias 3 -> 1
- net /GP10: track 24.6 -> 8.02 mm
- net +3.3V: track 218.5 -> 204.8 mm
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- removed copper zone on B.Cu, net +5V
- removed copper zone on F.Cu, net +5V
Other:
- outline, holes or cut-outs redrawn
- board text added: "- + A B"
- board text removed: "B A + -"
