File: picoControl/board/kicadV3.0/smallcontrol.kicad_sch (KiCad schematic)
At the start: 45 parts, among them J1 dynamixel, J10 OLED, J11 CSRF, J14 lineOut1, J15 grove I2C, J2 Audio1, J23 PowerIn, J24 grove GPIO / waveshare DDSM, J25 PowerIn, J26 grove GPIO / waveshare DDSM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

Commit message: update config.cpp system
Parts:
- added J16: grove Analog, Connector:NS-Tech_Grove_1x04_P2mm_Vertical, symbol Connector_Generic:Conn_01x04
- C1, C15, C2, C5, C8: footprint fab:C_1206 -> Capacitor_SMD:C_0603_1608Metric_Pad1.08x0.95mm_HandSolder
- J15, J24, J26: footprint Connectors:Grove_1x04 -> Connector:NS-Tech_Grove_1x04_P2mm_Vertical
- R1, R10, R2, R3, R4, R9: footprint fab:R_1206 -> Resistor_SMD:R_0603_1608Metric_Pad0.98x0.95mm_HandSolder
Connections:
- net +3.3V: now also J7.2 (Pin_2), R2.1, U1.8 (VCC), J16.2 (Pin_2); no longer J7.6 (Pin_6)
- net +5V: no longer R2.1, U1.8 (VCC)
- net 12Vfused: now also J1.3 (Pin_3); no longer J1.2 (Pin_2)
- net A: now also J1.2 (Pin_2); no longer J1.3 (Pin_3)
- net B: now also J1.1 (Pin_1); no longer J1.4 (Pin_4)
- net GND: now also J1.4 (Pin_4), J7.9 (Pin_9), J16.1 (Pin_1); no longer J1.1 (Pin_1), J7.5 (Pin_5)
- net GP10: no longer M1.20 (GP15)
- net GP15: now also M1.20 (GP15)
- net INA1: now also J7.5 (Pin_5); no longer J7.3 (Pin_3)
- net INA2: now also J7.7 (Pin_7); no longer J7.8 (Pin_8)
- net INB1: now also J7.6 (Pin_6); no longer J7.4 (Pin_4)
- net INB2: now also J7.8 (Pin_8); no longer J7.9 (Pin_9)
- net PWM1: now also J7.3 (Pin_3); no longer J7.2 (Pin_2)
- net PWM2: now also J7.4 (Pin_4); no longer J7.7 (Pin_7)
- net at M1.32 (GP27): now also J16.4 (Pin_4)
- net at M1.34 (GP28): now also J16.3 (Pin_3)
